File: 01_Cell_Module_Row1.kicad_sch (KiCad schematic)
At the start: 48 parts

Commit message: Convert pack to 14S with 7 NTC sensors, JST XH harness connectors, all-JLC BOM
- Schematic regenerated: 14 cells, 15-wire BMS sense on JST XH B15B-XH-A,
  7x 10k B3950 NTC saddles on JST XH B14B-XH-A, per-cell test loops and
  reverse-insertion indicator, power path with 5x20 fuse and M4 lugs.
- Fixes: HV zener was reversed, 4.7k/1206 HV LED resistor dissipated 0.68W
  (now 22k), 24V PPTCs on sense taps replaced with 60V MF-MSMF010-2,
  fuse-blown LED polarity corrected.
- Banana jacks (not stocked at LCSC) replaced by Keystone 5000/5001 loops.
- PCB re-laid out on the A4 (297x210) 4-layer outline: 8+6 cell columns,
  zones for cell links, sense routed on In1, NTC pairs on In2.
- ERC 0, DRC 0 (all severities), 0 unconnected, 0 schematic parity issues.
- Added Gerbers/drill zip, JLCPCB BOM + CPL, schematic PDF, renders, and the
  generator scripts in tools/.

Co-Authored-By: Claude Opus 5.5 <noreply@anthropic.com>
Claude-Session: https://claude.ai/code/session_01SDBUxKR8a94h5ECbt5NLbF
Parts:
- removed BT8: BH-18650-B5BA008, footprints:BH18650B1BA002, symbol Device:Battery_Cell
- removed D_REV_1, D_REV_2, D_REV_3, D_REV_4, D_REV_5, D_REV_6, D_REV_7, D_REV_8: 1N4148WS [C2128], Diode_SMD:D_SOD-323, symbol Device:D
- removed J_NEG_1, J_NEG_2, J_NEG_3, J_NEG_4, J_NEG_5, J_NEG_6, J_NEG_7, J_NEG_8: 575-8_BLK_4MM, Connector:Banana_Jack_1Pin, symbol Connector_Generic:Conn_01x01
- removed J_POS_1, J_POS_2, J_POS_3, J_POS_4, J_POS_5, J_POS_6, J_POS_7, J_POS_8: 575-4_RED_4MM, Connector:Banana_Jack_1Pin, symbol Connector_Generic:Conn_01x01
- removed LED_REV_1, LED_REV_2, LED_REV_3, LED_REV_4, LED_REV_5, LED_REV_6, LED_REV_7, LED_REV_8: KT-0805R [C2295], LED_SMD:LED_0805_2012Metric, symbol Device:LED
- removed R_REV_1, R_REV_2, R_REV_3, R_REV_4, R_REV_5, R_REV_6, R_REV_7, R_REV_8: 1k_1%_0805 [C17513], Resistor_SMD:R_0805_2012Metric, symbol Device:R
- added D_REV1, D_REV2, D_REV3, D_REV4, D_REV5, D_REV6, D_REV7: 1N4148WS, Diode_SMD:D_SOD-323, symbol Device:D
- added LED_REV1, LED_REV2, LED_REV3, LED_REV4, LED_REV5, LED_REV6, LED_REV7: RED, LED_SMD:LED_0805_2012Metric, symbol Device:LED
- added R_REV1, R_REV2, R_REV3, R_REV4, R_REV5, R_REV6, R_REV7: 1k, Resistor_SMD:R_0805_2012Metric, symbol Device:R
- added TP_N1, TP_N2, TP_N3, TP_N4, TP_N5, TP_N6, TP_N7: 5001 BLK, TestPoint:TestPoint_Keystone_5000-5004_Miniature, symbol Connector:TestPoint
- added TP_P1, TP_P2, TP_P3, TP_P4, TP_P5, TP_P6, TP_P7: 5000 RED, TestPoint:TestPoint_Keystone_5000-5004_Miniature, symbol Connector:TestPoint
- BT1, BT2, BT3, BT4, BT5, BT6, BT7: value BH-18650-B5BA008 -> 18650 holder; JLCPCB Part # C2988620 -> (none); MPN BH-18650-B5BA008 -> BH-18650-B1BA002; Manufacturer (none) -> MYOUNG
Connections:
- net CELL_1: now also D_REV1.1 (K), R_REV2.2, TP_N2.1, TP_P1.1
- net CELL_2: now also D_REV2.1 (K), R_REV3.2, TP_N3.1, TP_P2.1
- net CELL_3: now also D_REV3.1 (K), R_REV4.2, TP_N4.1, TP_P3.1
- net CELL_4: now also D_REV4.1 (K), R_REV5.2, TP_N5.1, TP_P4.1
- net CELL_5: now also D_REV5.1 (K), R_REV6.2, TP_N6.1, TP_P5.1
- net CELL_6: now also D_REV6.1 (K), R_REV7.2, TP_N7.1, TP_P6.1
- net CELL_7: now also D_REV7.1 (K), TP_P7.1
- net GND renamed PACK_NEG
- net PACK_NEG: now also R_REV1.2, TP_N1.1
- new net: LED_REV2.2 (A), R_REV2.1
- new net: LED_REV6.2 (A), R_REV6.1
- new net: LED_REV4.2 (A), R_REV4.1
- new net: LED_REV5.2 (A), R_REV5.1
- new net: D_REV5.2 (A), LED_REV5.1 (K)
- new net: D_REV2.2 (A), LED_REV2.1 (K)
- new net: D_REV1.2 (A), LED_REV1.1 (K)
- new net: LED_REV1.2 (A), R_REV1.1
- new net: D_REV7.2 (A), LED_REV7.1 (K)
- new net: D_REV6.2 (A), LED_REV6.1 (K)
- new net: D_REV3.2 (A), LED_REV3.1 (K)
- new net: LED_REV3.2 (A), R_REV3.1
- new net: LED_REV7.2 (A), R_REV7.1
- new net: D_REV4.2 (A), LED_REV4.1 (K)
Other:
- note added: "CELL 1"
- note added: "CELL 2"
- note added: "CELL 3"
- note added: "CELL 4"
- note added: "CELL 5"
- note added: "CELL 6"
- note added: "CELL 7"
- note added: "CELL MODULE A: CELLS 1 TO 7 Each cell: 18650 holder, red (+) / black (-) test loops, and a zero-drain reverse-insertion indicator (R -> LED -> 1N4148WS). It only conducts if the cell is fitted backwards, so it draws nothing in normal use."
- note removed: "CELL MODULE 1: CELLS 1 TO 8 (UPPER CARRIER) Symmetrical Layout &bull; Across-Cell Banana Jacks &bull; Zero-Drain Reverse Polarity Alert Triads"
- company: Antigravity Battery Engineering -> Battery Pack Breakout - 14S / A4
- title: CELL MODULE 1: CELLS 1 TO 8 (UPPER CARRIER) -> CELL MODULE A: CELLS 1 TO 7

Commit message: Make the board mirror-symmetric about its centre line
- NTCs: 3 per side in mirrored gaps, NTC4 on the centre line at the
  cell 7->8 bus (J2 pins 7/8); J2 pin 2n-1/2n = NTCn kept.
- Sense spine exactly symmetric: tap-7 PPTC and its bus line on the centre
  line, side buses mirrored, J1 fan symmetric.
- Per-cell LED strings: series order chosen per cell so mirrored twins use
  the same parts in the same places (function unchanged).
- TVS chain under J1 mirrored; the centre pair stands vertically either side
  of lane 7.
- HV indicator + pack TVS centred at J2's mirror position; top-band copper
  mirrored; 4 corner fiducials.
- tools/symcheck.py audits mirror partners: only J2, the HV block and the
  single PACK+ fuse (+ its LED) are one-of-a-kind.
- ERC 0, DRC 0, 0 unconnected, 0 parity; ACIR spread 0.08 %.

Co-Authored-By: Claude Opus 5.5 <noreply@anthropic.com>
Claude-Session: https://claude.ai/code/session_01SDBUxKR8a94h5ECbt5NLbF
Connections:
- net CELL_1: now also R_REV1.1; no longer D_REV1.1 (K)
- net CELL_2: now also D_REV3.2 (A); no longer R_REV3.2
- net CELL_3: now also R_REV3.1; no longer D_REV3.1 (K)
- net CELL_4: now also D_REV5.2 (A); no longer R_REV5.2
- net CELL_5: now also R_REV5.1; no longer D_REV5.1 (K)
- net CELL_6: now also D_REV7.2 (A); no longer R_REV7.2
- net CELL_7: now also R_REV7.1; no longer D_REV7.1 (K)
- net PACK_NEG: now also D_REV1.2 (A); no longer R_REV1.2
- net at LED_REV5.2 (A): now also D_REV5.1 (K); no longer R_REV5.1
- net at LED_REV5.1 (K): now also R_REV5.2; no longer D_REV5.2 (A)
- net at LED_REV1.1 (K): now also R_REV1.2; no longer D_REV1.2 (A)
- net at LED_REV1.2 (A): now also D_REV1.1 (K); no longer R_REV1.1
- net at LED_REV7.1 (K): now also R_REV7.2; no longer D_REV7.2 (A)
- net at LED_REV3.1 (K): now also R_REV3.2; no longer D_REV3.2 (A)
- net at LED_REV3.2 (A): now also D_REV3.1 (K); no longer R_REV3.1
- net at LED_REV7.2 (A): now also D_REV7.1 (K); no longer R_REV7.1
Other:
- moved on the sheet: D_REV1, D_REV3, D_REV5, D_REV7, R_REV1, R_REV3, R_REV5, R_REV7
