File: 02_Cell_Module_Row2.kicad_sch (KiCad schematic)
At the start: 48 parts

Commit message: Convert pack to 14S with 7 NTC sensors, JST XH harness connectors, all-JLC BOM
- Schematic regenerated: 14 cells, 15-wire BMS sense on JST XH B15B-XH-A,
  7x 10k B3950 NTC saddles on JST XH B14B-XH-A, per-cell test loops and
  reverse-insertion indicator, power path with 5x20 fuse and M4 lugs.
- Fixes: HV zener was reversed, 4.7k/1206 HV LED resistor dissipated 0.68W
  (now 22k), 24V PPTCs on sense taps replaced with 60V MF-MSMF010-2,
  fuse-blown LED polarity corrected.
- Banana jacks (not stocked at LCSC) replaced by Keystone 5000/5001 loops.
- PCB re-laid out on the A4 (297x210) 4-layer outline: 8+6 cell columns,
  zones for cell links, sense routed on In1, NTC pairs on In2.
- ERC 0, DRC 0 (all severities), 0 unconnected, 0 schematic parity issues.
- Added Gerbers/drill zip, JLCPCB BOM + CPL, schematic PDF, renders, and the
  generator scripts in tools/.

Co-Authored-By: Claude Opus 5.5 <noreply@anthropic.com>
Claude-Session: https://claude.ai/code/session_01SDBUxKR8a94h5ECbt5NLbF
Parts:
- removed BT15, BT16: BH-18650-B5BA008, footprints:BH18650B1BA002, symbol Device:Battery_Cell
- removed D_REV_10, D_REV_11, D_REV_12, D_REV_13, D_REV_14, D_REV_15, D_REV_16, D_REV_9: 1N4148WS [C2128], Diode_SMD:D_SOD-323, symbol Device:D
- removed J_NEG_10, J_NEG_11, J_NEG_12, J_NEG_13, J_NEG_14, J_NEG_15, J_NEG_16, J_NEG_9: 575-8_BLK_4MM, Connector:Banana_Jack_1Pin, symbol Connector_Generic:Conn_01x01
- removed J_POS_10, J_POS_11, J_POS_12, J_POS_13, J_POS_14, J_POS_15, J_POS_16, J_POS_9: 575-4_RED_4MM, Connector:Banana_Jack_1Pin, symbol Connector_Generic:Conn_01x01
- removed LED_REV_10, LED_REV_11, LED_REV_12, LED_REV_13, LED_REV_14, LED_REV_15, LED_REV_16, LED_REV_9: KT-0805R [C2295], LED_SMD:LED_0805_2012Metric, symbol Device:LED
- removed R_REV_10, R_REV_11, R_REV_12, R_REV_13, R_REV_14, R_REV_15, R_REV_16, R_REV_9: 1k_1%_0805 [C17513], Resistor_SMD:R_0805_2012Metric, symbol Device:R
- added BT8: 18650 holder, footprints:BH18650B1BA002, symbol Device:Battery_Cell
- added D_REV10, D_REV11, D_REV12, D_REV13, D_REV14, D_REV8, D_REV9: 1N4148WS, Diode_SMD:D_SOD-323, symbol Device:D
- added LED_REV10, LED_REV11, LED_REV12, LED_REV13, LED_REV14, LED_REV8, LED_REV9: RED, LED_SMD:LED_0805_2012Metric, symbol Device:LED
- added R_REV10, R_REV11, R_REV12, R_REV13, R_REV14, R_REV8, R_REV9: 1k, Resistor_SMD:R_0805_2012Metric, symbol Device:R
- added TP_N10, TP_N11, TP_N12, TP_N13, TP_N14, TP_N8, TP_N9: 5001 BLK, TestPoint:TestPoint_Keystone_5000-5004_Miniature, symbol Connector:TestPoint
- added TP_P10, TP_P11, TP_P12, TP_P13, TP_P14, TP_P8, TP_P9: 5000 RED, TestPoint:TestPoint_Keystone_5000-5004_Miniature, symbol Connector:TestPoint
- BT10, BT11, BT12, BT13, BT14, BT9: value BH-18650-B5BA008 -> 18650 holder; JLCPCB Part # C2988620 -> (none); MPN BH-18650-B5BA008 -> BH-18650-B1BA002; Manufacturer (none) -> MYOUNG
Connections:
- net CELL_10: now also D_REV10.1 (K), R_REV11.2, TP_N11.1, TP_P10.1
- net CELL_11: now also D_REV11.1 (K), R_REV12.2, TP_N12.1, TP_P11.1
- net CELL_12: now also D_REV12.1 (K), R_REV13.2, TP_N13.1, TP_P12.1
- net CELL_13: now also D_REV13.1 (K), R_REV14.2, TP_N14.1, TP_P13.1
- net CELL_8: now also BT8.1 (+), D_REV8.1 (K), R_REV9.2, TP_N9.1, TP_P8.1
- net CELL_9: now also D_REV9.1 (K), R_REV10.2, TP_N10.1, TP_P9.1
- net CELL_14 renamed CELL_14_UNFUSED
- net CELL_14_UNFUSED: now also D_REV14.1 (K), TP_P14.1
- new net: D_REV10.2 (A), LED_REV10.1 (K)
- new net: LED_REV10.2 (A), R_REV10.1
- new net: LED_REV14.2 (A), R_REV14.1
- new net: D_REV9.2 (A), LED_REV9.1 (K)
- new net: LED_REV9.2 (A), R_REV9.1
- new net: LED_REV12.2 (A), R_REV12.1
- new net: D_REV14.2 (A), LED_REV14.1 (K)
- new net: D_REV13.2 (A), LED_REV13.1 (K)
- new net: D_REV12.2 (A), LED_REV12.1 (K)
- new net: LED_REV13.2 (A), R_REV13.1
- new net: D_REV11.2 (A), LED_REV11.1 (K)
- new net: LED_REV11.2 (A), R_REV11.1
- new net: D_REV8.2 (A), LED_REV8.1 (K)
- new net: LED_REV8.2 (A), R_REV8.1
- new net CELL_7: BT8.2 (-), R_REV8.2, TP_N8.1
Other:
- note added: "CELL 10"
- note added: "CELL 11"
- note added: "CELL 12"
- note added: "CELL 13"
- note added: "CELL 14"
- note added: "CELL 8"
- note added: "CELL 9"
- note added: "CELL MODULE B: CELLS 8 TO 14 Each cell: 18650 holder, red (+) / black (-) test loops, and a zero-drain reverse-insertion indicator (R -> LED -> 1N4148WS). It only conducts if the cell is fitted backwards, so it draws nothing in normal use."
- note removed: "CELL MODULE 2: CELLS 9 TO 16 (LOWER CARRIER) Symmetrical Layout &bull; Across-Cell Banana Jacks &bull; Zero-Drain Reverse Polarity Alert Triads"
- company: Antigravity Battery Engineering -> Battery Pack Breakout - 14S / A4
- title: CELL MODULE 2: CELLS 9 TO 16 (LOWER CARRIER) -> CELL MODULE B: CELLS 8 TO 14

Commit message: Make the board mirror-symmetric about its centre line
- NTCs: 3 per side in mirrored gaps, NTC4 on the centre line at the
  cell 7->8 bus (J2 pins 7/8); J2 pin 2n-1/2n = NTCn kept.
- Sense spine exactly symmetric: tap-7 PPTC and its bus line on the centre
  line, side buses mirrored, J1 fan symmetric.
- Per-cell LED strings: series order chosen per cell so mirrored twins use
  the same parts in the same places (function unchanged).
- TVS chain under J1 mirrored; the centre pair stands vertically either side
  of lane 7.
- HV indicator + pack TVS centred at J2's mirror position; top-band copper
  mirrored; 4 corner fiducials.
- tools/symcheck.py audits mirror partners: only J2, the HV block and the
  single PACK+ fuse (+ its LED) are one-of-a-kind.
- ERC 0, DRC 0, 0 unconnected, 0 parity; ACIR spread 0.08 %.

Co-Authored-By: Claude Opus 5.5 <noreply@anthropic.com>
Claude-Session: https://claude.ai/code/session_01SDBUxKR8a94h5ECbt5NLbF
Connections:
- net CELL_10: now also D_REV11.2 (A); no longer R_REV11.2
- net CELL_11: now also R_REV11.1; no longer D_REV11.1 (K)
- net CELL_12: now also D_REV13.2 (A); no longer R_REV13.2
- net CELL_13: now also R_REV13.1; no longer D_REV13.1 (K)
- net CELL_8: now also D_REV9.2 (A); no longer R_REV9.2
- net CELL_9: now also R_REV9.1; no longer D_REV9.1 (K)
- net at LED_REV9.1 (K): now also R_REV9.2; no longer D_REV9.2 (A)
- net at LED_REV9.2 (A): now also D_REV9.1 (K); no longer R_REV9.1
- net at LED_REV13.1 (K): now also R_REV13.2; no longer D_REV13.2 (A)
- net at LED_REV13.2 (A): now also D_REV13.1 (K); no longer R_REV13.1
- net at LED_REV11.1 (K): now also R_REV11.2; no longer D_REV11.2 (A)
- net at LED_REV11.2 (A): now also D_REV11.1 (K); no longer R_REV11.1
Other:
- moved on the sheet: D_REV11, D_REV13, D_REV9, R_REV11, R_REV13, R_REV9
Changed lines of the file:
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@@
 	)
 	(symbol
-		(lib_id "Device:D")
-		(at 109.22 73.66 270)
+		(lib_id "Device:R")
+		(at 109.22 73.66 0)
 		(unit 1)
 		(body_style 1)
@@
 		(in_pos_files yes)
 		(dnp no)
-		(property "Reference" "D_REV9"
-			(at 111.76 72.39 90)
+		(property "Reference" "R_REV9"
+			(at 111.76 72.39 0)
 			(show_name no)
 			(do_not_autoplace no)
@@
 			)
 		)
-		(property "Value" "1N4148WS"
-			(at 111.76 74.93 90)
+		(property "Value" "1k"
+			(at 111.76 74.93 0)
 			(show_name no)
 			(do_not_autoplace no)
@@
 			)
 		)
-		(property "Footprint" "Diode_SMD:D_SOD-323"
+		(property "Footprint" "Resistor_SMD:R_0805_2012Metric"
 			(at 109.22 73.66 0)
 			(hide yes)
@@
 			)
 		)
-		(property "Description" "75V 150mA switching diode, blocks LED reverse bias"
+		(property "Description" "1k 1% 0805 - reverse-cell LED limit"
 			(at 109.22 73.66 0)
 			(hide yes)
@@
 			)
 		)
-		(property "LCSC" "C2128"
+		(property "LCSC" "C17513"
 			(at 109.22 73.66 0)
 			(hide yes)
@@
 			)
 		)
-		(property "MPN" "1N4148WS"
+		(property "MPN" "0805W8F1001T5E"
 			(at 109.22 73.66 0)
 			(hide yes)
@@
 			)
 		)
-		(property "Manufacturer" "CJ"
+		(property "Manufacturer" "UNI-ROYAL"
 			(at 109.22 73.66 0)
 			(hide yes)
@@
 			(project "BatteryPack_16S_A4_Breakout"
 				(path "/00000000-0000-0000-0000-000000000001/00000000-0000-0000-0000-000000000003"
-					(reference "D_REV9")
+					(reference "R_REV9")
 					(unit 1)
 				)
@@
 	)
 	(symbol
-		(lib_id "Device:R")
-		(at 109.22 104.14 0)
+		(lib_id "Device:D")
+		(at 109.22 104.14 270)
 		(unit 1)
 		(body_style 1)
@@
 		(in_pos_files yes)
 		(dnp no)
-		(property "Reference" "R_REV9"
-			(at 111.76 102.87 0)
+		(property "Reference" "D_REV9"
+			(at 111.76 102.87 90)
 			(show_name no)
 			(do_not_autoplace no)
@@
 			)
 		)
-		(property "Value" "1k"
-			(at 111.76 105.41 0)
+		(property "Value" "1N4148WS"
+			(at 111.76 105.41 90)
 			(show_name no)
 			(do_not_autoplace no)
@@
 			)
 		)
-		(property "Footprint" "Resistor_SMD:R_0805_2012Metric"
+		(property "Footprint" "Diode_SMD:D_SOD-323"
 			(at 109.22 104.14 0)
 			(hide yes)
@@
 			)
 		)
-		(property "Description" "1k 1% 0805 - reverse-cell LED limit"
+		(property "Description" "75V 150mA switching diode, blocks LED reverse bias"
 			(at 109.22 104.14 0)
 			(hide yes)
@@
 			)
 		)
-		(property "LCSC" "C17513"
+		(property "LCSC" "C2128"
 			(at 109.22 104.14 0)
 			(hide yes)
@@
 			)
 		)
-		(property "MPN" "0805W8F1001T5E"
+		(property "MPN" "1N4148WS"
 			(at 109.22 104.14 0)
 			(hide yes)
@@
 			)
 		)
-		(property "Manufacturer" "UNI-ROYAL"
+		(property "Manufacturer" "CJ"
 			(at 109.22 104.14 0)
 			(hide yes)
@@
 			(project "BatteryPack_16S_A4_Breakout"
 				(path "/00000000-0000-0000-0000-000000000001/00000000-0000-0000-0000-000000000003"
-					(reference "R_REV9")
+					(reference "D_REV9")
 					(unit 1)
 				)
@@
 	)
 	(symbol
-		(lib_id "Device:D")
-		(at 215.9 73.66 270)
+		(lib_id "Device:R")
+		(at 215.9 73.66 0)
 		(unit 1)
 		(body_style 1)
@@
 		(in_pos_files yes)
 		(dnp no)
-		(property "Reference" "D_REV11"
-			(at 218.44 72.39 90)
+		(property "Reference" "R_REV11"
+			(at 218.44 72.39 0)
 			(show_name no)
 			(do_not_autoplace no)
@@
 			)
 		)
-		(property "Value" "1N4148WS"
-			(at 218.44 74.93 90)
+		(property "Value" "1k"
+			(at 218.44 74.93 0)
 			(show_name no)
 			(do_not_autoplace no)
@@
 			)
 		)
-		(property "Footprint" "Diode_SMD:D_SOD-323"
+		(property "Footprint" "Resistor_SMD:R_0805_2012Metric"
 			(at 215.9 73.66 0)
 			(hide yes)
@@
 			)
 		)
-		(property "Description" "75V 150mA switching diode, blocks LED reverse bias"
+		(property "Description" "1k 1% 0805 - reverse-cell LED limit"
 			(at 215.9 73.66 0)
 			(hide yes)
@@
 			)
 		)
-		(property "LCSC" "C2128"
+		(property "LCSC" "C17513"
 			(at 215.9 73.66 0)
 			(hide yes)
@@
 			)
 		)
-		(property "MPN" "1N4148WS"
+		(property "MPN" "0805W8F1001T5E"
 			(at 215.9 73.66 0)
 			(hide yes)
@@
 			)
 		)
-		(property "Manufacturer" "CJ"
+		(property "Manufacturer" "UNI-ROYAL"
 			(at 215.9 73.66 0)
 			(hide yes)
@@
 			(project "BatteryPack_16S_A4_Breakout"
 				(path "/00000000-0000-0000-0000-000000000001/00000000-0000-0000-0000-000000000003"
-					(reference "D_REV11")
+					(reference "R_REV11")
 					(unit 1)
 				)
@@
 	)
 	(symbol
-		(lib_id "Device:R")
-		(at 215.9 104.14 0)
+		(lib_id "Device:D")
+		(at 215.9 104.14 270)
 		(unit 1)
 		(body_style 1)
@@
 		(in_pos_files yes)
 		(dnp no)
-		(property "Reference" "R_REV11"
-			(at 218.44 102.87 0)
+		(property "Reference" "D_REV11"
+			(at 218.44 102.87 90)
 			(show_name no)
 			(do_not_autoplace no)
@@
 			)
 		)
-		(property "Value" "1k"
-			(at 218.44 105.41 0)
+		(property "Value" "1N4148WS"
+			(at 218.44 105.41 90)
 			(show_name no)
 			(do_not_autoplace no)
@@
 			)
 		)
-		(property "Footprint" "Resistor_SMD:R_0805_2012Metric"
+		(property "Footprint" "Diode_SMD:D_SOD-323"
 			(at 215.9 104.14 0)
 			(hide yes)
@@
 			)
 		)
-		(property "Description" "1k 1% 0805 - reverse-cell LED limit"
+		(property "Description" "75V 150mA switching diode, blocks LED reverse bias"
 			(at 215.9 104.14 0)
 			(hide yes)
@@
 			)
 		)
-		(property "LCSC" "C17513"
+		(property "LCSC" "C2128"
 			(at 215.9 104.14 0)
 			(hide yes)
@@
 			)
 		)
-		(property "MPN" "0805W8F1001T5E"
+		(property "MPN" "1N4148WS"
 			(at 215.9 104.14 0)
 			(hide yes)
@@
 			)
 		)
-		(property "Manufacturer" "UNI-ROYAL"
+		(property "Manufacturer" "CJ"
 			(at 215.9 104.14 0)
 			(hide yes)
@@
 			(project "BatteryPack_16S_A4_Breakout"
 				(path "/00000000-0000-0000-0000-000000000001/00000000-0000-0000-0000-000000000003"
-					(reference "R_REV11")
+					(reference "D_REV11")
 					(unit 1)
 				)
@@
 	)
 	(symbol
-		(lib_id "Device:D")
-		(at 322.58 73.66 270)
+		(lib_id "Device:R")
+		(at 322.58 73.66 0)
 		(unit 1)
 		(body_style 1)
@@
 		(in_pos_files yes)
 		(dnp no)
-		(property "Reference" "D_REV13"
-			(at 325.12 72.39 90)
+		(property "Reference" "R_REV13"
+			(at 325.12 72.39 0)
 			(show_name no)
 			(do_not_autoplace no)
@@
 			)
 		)
-		(property "Value" "1N4148WS"
-			(at 325.12 74.93 90)
+		(property "Value" "1k"
+			(at 325.12 74.93 0)
 			(show_name no)
 			(do_not_autoplace no)
@@
 			)
 		)
-		(property "Footprint" "Diode_SMD:D_SOD-323"
+		(property "Footprint" "Resistor_SMD:R_0805_2012Metric"
 			(at 322.58 73.66 0)
 			(hide yes)
@@
 			)
 		)
-		(property "Description" "75V 150mA switching diode, blocks LED reverse bias"
+		(property "Description" "1k 1% 0805 - reverse-cell LED limit"
 			(at 322.58 73.66 0)
 			(hide yes)
@@
 			)
 		)
-		(property "LCSC" "C2128"
+		(property "LCSC" "C17513"
 			(at 322.58 73.66 0)
 			(hide yes)
@@
 			)
 		)
-		(property "MPN" "1N4148WS"
+		(property "MPN" "0805W8F1001T5E"
 			(at 322.58 73.66 0)
 			(hide yes)
@@
 			)
 		)
-		(property "Manufacturer" "CJ"
+		(property "Manufacturer" "UNI-ROYAL"
 			(at 322.58 73.66 0)
 			(hide yes)
@@
 			(project "BatteryPack_16S_A4_Breakout"
 				(path "/00000000-0000-0000-0000-000000000001/00000000-0000-0000-0000-000000000003"
-					(reference "D_REV13")
+					(reference "R_REV13")
 					(unit 1)
 				)
@@
 	)
 	(symbol
-		(lib_id "Device:R")
-		(at 322.58 104.14 0)
+		(lib_id "Device:D")
+		(at 322.58 104.14 270)
 		(unit 1)
 		(body_style 1)
@@
 		(in_pos_files yes)
 		(dnp no)
-		(property "Reference" "R_REV13"
-			(at 325.12 102.87 0)
+		(property "Reference" "D_REV13"
+			(at 325.12 102.87 90)
 			(show_name no)
 			(do_not_autoplace no)
@@
 			)
 		)
-		(property "Value" "1k"
-			(at 325.12 105.41 0)
+		(property "Value" "1N4148WS"
+			(at 325.12 105.41 90)
 			(show_name no)
 			(do_not_autoplace no)
@@
 			)
 		)
-		(property "Footprint" "Resistor_SMD:R_0805_2012Metric"
+		(property "Footprint" "Diode_SMD:D_SOD-323"
 			(at 322.58 104.14 0)
 			(hide yes)
@@
 			)
 		)
-		(property "Description" "1k 1% 0805 - reverse-cell LED limit"
+		(property "Description" "75V 150mA switching diode, blocks LED reverse bias"
 			(at 322.58 104.14 0)
 			(hide yes)
@@
 			)
 		)
-		(property "LCSC" "C17513"
+		(property "LCSC" "C2128"
 			(at 322.58 104.14 0)
 			(hide yes)
@@
 			)
 		)
-		(property "MPN" "0805W8F1001T5E"
+		(property "MPN" "1N4148WS"
 			(at 322.58 104.14 0)
 			(hide yes)
@@
 			)
 		)
-		(property "Manufacturer" "UNI-ROYAL"
+		(property "Manufacturer" "CJ"
 			(at 322.58 104.14 0)
 			(hide yes)
@@
 			(project "BatteryPack_16S_A4_Breakout"
 				(path "/00000000-0000-0000-0000-000000000001/00000000-0000-0000-0000-000000000003"
-					(reference "R_REV13")
+					(reference "D_REV13")
 					(unit 1)
 				)
