File: BatteryPack_16S_A4_Breakout.kicad_pcb (KiCad board)
At the start: 4 copper layers, 297 x 210 mm, 165 parts, among them J1 HDR-1X17_2.54mm [C22549], J2 S16B-XH-A [C157933], J3 T44009_M4_POS [C481463], J4 T44009_M4_GND [C481463]

Commit message: Convert pack to 14S with 7 NTC sensors, JST XH harness connectors, all-JLC BOM
- Schematic regenerated: 14 cells, 15-wire BMS sense on JST XH B15B-XH-A,
  7x 10k B3950 NTC saddles on JST XH B14B-XH-A, per-cell test loops and
  reverse-insertion indicator, power path with 5x20 fuse and M4 lugs.
- Fixes: HV zener was reversed, 4.7k/1206 HV LED resistor dissipated 0.68W
  (now 22k), 24V PPTCs on sense taps replaced with 60V MF-MSMF010-2,
  fuse-blown LED polarity corrected.
- Banana jacks (not stocked at LCSC) replaced by Keystone 5000/5001 loops.
- PCB re-laid out on the A4 (297x210) 4-layer outline: 8+6 cell columns,
  zones for cell links, sense routed on In1, NTC pairs on In2.
- ERC 0, DRC 0 (all severities), 0 unconnected, 0 schematic parity issues.
- Added Gerbers/drill zip, JLCPCB BOM + CPL, schematic PDF, renders, and the
  generator scripts in tools/.

Co-Authored-By: Claude Opus 5.5 <noreply@anthropic.com>
Claude-Session: https://claude.ai/code/session_01SDBUxKR8a94h5ECbt5NLbF
Parts:
- removed BT15, BT16: BH-18650-B5BA008, footprints:BH18650B1BA002
- removed D_FUSE_BLOWN1: KT-0805Y_AMBER [C2296], LED_SMD:LED_0805_2012Metric
- removed D_REV_1, D_REV_10, D_REV_11, D_REV_12, D_REV_13, D_REV_14, D_REV_15, D_REV_16, D_REV_2, D_REV_3, D_REV_4, D_REV_5, D_REV_6, D_REV_7, D_REV_8, D_REV_9: 1N4148WS [C2128], Diode_SMD:D_SOD-323
- removed D_TVS15, D_TVS16: SMAJ5.0CA [C266332], Diode_SMD:D_SMA
- removed D_ZENER_HV1: BZX84C43_43V [C7093918], Package_TO_SOT_SMD:SOT-23
- removed F_PTC16, F_PTC17: 1206L020YR_200mA [C207035], Resistor_SMD:R_1206_3216Metric
- removed J_NEG_1, J_NEG_10, J_NEG_11, J_NEG_12, J_NEG_13, J_NEG_14, J_NEG_15, J_NEG_16, J_NEG_2, J_NEG_3, J_NEG_4, J_NEG_5, J_NEG_6, J_NEG_7, J_NEG_8, J_NEG_9: 575-8_BLK_4MM, Connector:Banana_Jack_1Pin
- removed J_POS_1, J_POS_10, J_POS_11, J_POS_12, J_POS_13, J_POS_14, J_POS_15, J_POS_16, J_POS_2, J_POS_3, J_POS_4, J_POS_5, J_POS_6, J_POS_7, J_POS_8, J_POS_9: 575-4_RED_4MM, Connector:Banana_Jack_1Pin
- removed LED_REV_1, LED_REV_10, LED_REV_11, LED_REV_12, LED_REV_13, LED_REV_14, LED_REV_15, LED_REV_16, LED_REV_2, LED_REV_3, LED_REV_4, LED_REV_5, LED_REV_6, LED_REV_7, LED_REV_8, LED_REV_9: KT-0805R [C2295], LED_SMD:LED_0805_2012Metric
- removed R_FUSE_BLOWN1: 10k_1%_1206 [C17902], Resistor_SMD:R_1206_3216Metric
- removed R_REV_1, R_REV_10, R_REV_11, R_REV_12, R_REV_13, R_REV_14, R_REV_15, R_REV_16, R_REV_2, R_REV_3, R_REV_4, R_REV_5, R_REV_6, R_REV_7, R_REV_8, R_REV_9: 1k_1%_0805 [C17513], Resistor_SMD:R_0805_2012Metric
- removed TH8: MF52A103J3950_10k [C123378], Resistor_THT:R_Axial_DIN0204_L3.6mm_D1.6mm_P2.54mm_Vertical
- removed TP_10S1, TP_14S1, TP_16S1, TP_7S1: Keystone_5000_RED [C5199900], TestPoint:TestPoint_Keystone_5000-5004_Miniature
- removed TP_GND1: Keystone_5001_BLK [C238122], TestPoint:TestPoint_Keystone_5000-5004_Miniature
- added D_HV1: BZX84C43, Package_TO_SOT_SMD:SOT-23, F.Cu at (134.0, 36.1)
- added D_REV1: 1N4148WS, Diode_SMD:D_SOD-323, F.Cu at (11.0, 21.5)
- added D_REV10: 1N4148WS, Diode_SMD:D_SOD-323, F.Cu at (286.0, 160.3)
- added D_REV11: 1N4148WS, Diode_SMD:D_SOD-323, F.Cu at (286.0, 139.0)
- added D_REV12: 1N4148WS, Diode_SMD:D_SOD-323, F.Cu at (286.0, 110.7)
- added D_REV13: 1N4148WS, Diode_SMD:D_SOD-323, F.Cu at (286.0, 89.4)
- added D_REV14: 1N4148WS, Diode_SMD:D_SOD-323, F.Cu at (286.0, 61.1)
- added D_REV2: 1N4148WS, Diode_SMD:D_SOD-323, F.Cu at (11.0, 49.8)
- added D_REV3: 1N4148WS, Diode_SMD:D_SOD-323, F.Cu at (11.0, 71.1)
- added D_REV4: 1N4148WS, Diode_SMD:D_SOD-323, F.Cu at (11.0, 99.4)
- added D_REV5: 1N4148WS, Diode_SMD:D_SOD-323, F.Cu at (11.0, 120.7)
- added D_REV6: 1N4148WS, Diode_SMD:D_SOD-323, F.Cu at (11.0, 149.0)
- added D_REV7: 1N4148WS, Diode_SMD:D_SOD-323, F.Cu at (11.0, 170.3)
- added D_REV8: 1N4148WS, Diode_SMD:D_SOD-323, F.Cu at (11.0, 198.6)
- added D_REV9: 1N4148WS, Diode_SMD:D_SOD-323, F.Cu at (286.0, 188.6)
- added LED_FB1: AMBER, LED_SMD:LED_0805_2012Metric, F.Cu at (212.3, 49.5)
- added LED_REV1: RED, LED_SMD:LED_0805_2012Metric, F.Cu at (11.0, 16.5)
- added LED_REV10: RED, LED_SMD:LED_0805_2012Metric, F.Cu at (286.0, 165.3)
- added LED_REV11: RED, LED_SMD:LED_0805_2012Metric, F.Cu at (286.0, 144.0)
- added LED_REV12: RED, LED_SMD:LED_0805_2012Metric, F.Cu at (286.0, 115.7)
- added LED_REV13: RED, LED_SMD:LED_0805_2012Metric, F.Cu at (286.0, 94.4)
- added LED_REV14: RED, LED_SMD:LED_0805_2012Metric, F.Cu at (286.0, 66.1)
- added LED_REV2: RED, LED_SMD:LED_0805_2012Metric, F.Cu at (11.0, 44.8)
- added LED_REV3: RED, LED_SMD:LED_0805_2012Metric, F.Cu at (11.0, 66.1)
- added LED_REV4: RED, LED_SMD:LED_0805_2012Metric, F.Cu at (11.0, 94.4)
- added LED_REV5: RED, LED_SMD:LED_0805_2012Metric, F.Cu at (11.0, 115.7)
- added LED_REV6: RED, LED_SMD:LED_0805_2012Metric, F.Cu at (11.0, 144.0)
- added LED_REV7: RED, LED_SMD:LED_0805_2012Metric, F.Cu at (11.0, 165.3)
- added LED_REV8: RED, LED_SMD:LED_0805_2012Metric, F.Cu at (11.0, 193.6)
- added LED_REV9: RED, LED_SMD:LED_0805_2012Metric, F.Cu at (286.0, 193.6)
- added R_FB1: 47k, Resistor_SMD:R_0805_2012Metric, F.Cu at (208.5, 49.5)
- added R_REV1: 1k, Resistor_SMD:R_0805_2012Metric, F.Cu at (11.0, 11.5)
- added R_REV10: 1k, Resistor_SMD:R_0805_2012Metric, F.Cu at (286.0, 170.3)
- added R_REV11: 1k, Resistor_SMD:R_0805_2012Metric, F.Cu at (286.0, 149.0)
- added R_REV12: 1k, Resistor_SMD:R_0805_2012Metric, F.Cu at (286.0, 120.7)
- added R_REV13: 1k, Resistor_SMD:R_0805_2012Metric, F.Cu at (286.0, 99.4)
- added R_REV14: 1k, Resistor_SMD:R_0805_2012Metric, F.Cu at (286.0, 71.1)
- added R_REV2: 1k, Resistor_SMD:R_0805_2012Metric, F.Cu at (11.0, 39.8)
- added R_REV3: 1k, Resistor_SMD:R_0805_2012Metric, F.Cu at (11.0, 61.1)
- added R_REV4: 1k, Resistor_SMD:R_0805_2012Metric, F.Cu at (11.0, 89.4)
- added R_REV5: 1k, Resistor_SMD:R_0805_2012Metric, F.Cu at (11.0, 110.7)
- added R_REV6: 1k, Resistor_SMD:R_0805_2012Metric, F.Cu at (11.0, 139.0)
- added R_REV7: 1k, Resistor_SMD:R_0805_2012Metric, F.Cu at (11.0, 160.3)
- added R_REV8: 1k, Resistor_SMD:R_0805_2012Metric, F.Cu at (11.0, 188.6)
- added R_REV9: 1k, Resistor_SMD:R_0805_2012Metric, F.Cu at (286.0, 198.6)
- added TP_N1: 5001 BLK, TestPoint:TestPoint_Keystone_5000-5004_Miniature, F.Cu at (4.60, 11.0)
- added TP_N10: 5001 BLK, TestPoint:TestPoint_Keystone_5000-5004_Miniature, F.Cu at (292.4, 170.8)
- added TP_N11: 5001 BLK, TestPoint:TestPoint_Keystone_5000-5004_Miniature, F.Cu at (292.4, 149.5)
- added TP_N12: 5001 BLK, TestPoint:TestPoint_Keystone_5000-5004_Miniature, F.Cu at (292.4, 121.2)
- added TP_N13: 5001 BLK, TestPoint:TestPoint_Keystone_5000-5004_Miniature, F.Cu at (292.4, 99.9)
- added TP_N14: 5001 BLK, TestPoint:TestPoint_Keystone_5000-5004_Miniature, F.Cu at (292.4, 71.6)
- added TP_N2: 5001 BLK, TestPoint:TestPoint_Keystone_5000-5004_Miniature, F.Cu at (4.60, 39.3)
- added TP_N3: 5001 BLK, TestPoint:TestPoint_Keystone_5000-5004_Miniature, F.Cu at (4.60, 60.6)
- added TP_N4: 5001 BLK, TestPoint:TestPoint_Keystone_5000-5004_Miniature, F.Cu at (4.60, 88.9)
- added TP_N5: 5001 BLK, TestPoint:TestPoint_Keystone_5000-5004_Miniature, F.Cu at (4.60, 110.2)
- added TP_N6: 5001 BLK, TestPoint:TestPoint_Keystone_5000-5004_Miniature, F.Cu at (4.60, 138.5)
- added TP_N7: 5001 BLK, TestPoint:TestPoint_Keystone_5000-5004_Miniature, F.Cu at (4.60, 159.8)
- added TP_N8: 5001 BLK, TestPoint:TestPoint_Keystone_5000-5004_Miniature, F.Cu at (4.60, 188.1)
- added TP_N9: 5001 BLK, TestPoint:TestPoint_Keystone_5000-5004_Miniature, F.Cu at (292.4, 199.1)
- added TP_P1: 5000 RED, TestPoint:TestPoint_Keystone_5000-5004_Miniature, F.Cu at (4.60, 22.0)
- added TP_P10: 5000 RED, TestPoint:TestPoint_Keystone_5000-5004_Miniature, F.Cu at (292.4, 159.8)
- added TP_P11: 5000 RED, TestPoint:TestPoint_Keystone_5000-5004_Miniature, F.Cu at (292.4, 138.5)
- added TP_P12: 5000 RED, TestPoint:TestPoint_Keystone_5000-5004_Miniature, F.Cu at (292.4, 110.2)
- added TP_P13: 5000 RED, TestPoint:TestPoint_Keystone_5000-5004_Miniature, F.Cu at (292.4, 88.9)
- added TP_P14: 5000 RED, TestPoint:TestPoint_Keystone_5000-5004_Miniature, F.Cu at (292.4, 60.6)
- added TP_P2: 5000 RED, TestPoint:TestPoint_Keystone_5000-5004_Miniature, F.Cu at (4.60, 50.3)
- added TP_P3: 5000 RED, TestPoint:TestPoint_Keystone_5000-5004_Miniature, F.Cu at (4.60, 71.6)
- added TP_P4: 5000 RED, TestPoint:TestPoint_Keystone_5000-5004_Miniature, F.Cu at (4.60, 99.9)
- added TP_P5: 5000 RED, TestPoint:TestPoint_Keystone_5000-5004_Miniature, F.Cu at (4.60, 121.2)
- added TP_P6: 5000 RED, TestPoint:TestPoint_Keystone_5000-5004_Miniature, F.Cu at (4.60, 149.5)
- added TP_P7: 5000 RED, TestPoint:TestPoint_Keystone_5000-5004_Miniature, F.Cu at (4.60, 170.8)
- added TP_P8: 5000 RED, TestPoint:TestPoint_Keystone_5000-5004_Miniature, F.Cu at (4.60, 199.1)
- added TP_P9: 5000 RED, TestPoint:TestPoint_Keystone_5000-5004_Miniature, F.Cu at (292.4, 188.1)
- BT1, BT10, BT11, BT12, BT13, BT14, BT2, BT3, BT4, BT5, BT6, BT7, BT8, BT9: value BH-18650-B5BA008 -> 18650 holder
- D_TVS1, D_TVS10, D_TVS11, D_TVS12, D_TVS13, D_TVS14, D_TVS2, D_TVS3, D_TVS4, D_TVS5, D_TVS6, D_TVS7, D_TVS8, D_TVS9: value SMAJ5.0CA [C266332] -> SMAJ5.0CA
- D_TVS_MAIN1: value SMCJ70CA_1500W [C1976987] -> SMCJ70CA
- F1: value FH1-200CK-B_20A [C268205] -> 5x20 holder, fit 10A
- FID1, FID2, FID3: value Fiducial_1mm -> Fiducial
- F_PTC1, F_PTC10, F_PTC11, F_PTC12, F_PTC13, F_PTC14, F_PTC15, F_PTC2, F_PTC3, F_PTC4, F_PTC5, F_PTC6, F_PTC7, F_PTC8, F_PTC9: value 1206L020YR_200mA [C207035] -> MF-MSMF010-2 60V/0.1A; footprint Resistor_SMD:R_1206_3216Metric -> Fuse:Fuse_1812_4532Metric
- H1, H2, H3, H4, H5, H6: value M3_ISOLATED_HOLE -> M3 ISO7380
- J1: value HDR-1X17_2.54mm [C22549] -> B15B-XH-A; footprint Connector_PinHeader_2.54mm:PinHeader_1x17_P2.54mm_Horizontal -> Connector_JST:JST_XH_B15B-XH-A_1x15_P2.50mm_Vertical
- J2: value S16B-XH-A [C157933] -> B14B-XH-A; footprint Connector_JST:JST_XH_S16B-XH-A_1x16_P2.50mm_Horizontal -> Connector_JST:JST_XH_B14B-XH-A_1x14_P2.50mm_Vertical
- J3: value T44009_M4_POS [C481463] -> PACK+ M4
- J4: value T44009_M4_GND [C481463] -> PACK- M4
- LED_HV1: value KT-0805R_HV [C2295] -> RED
- Q_HV1: value MMBTA42_300V [C8515] -> MMBTA42
- R_HV_BASE1: value 10k_1%_0805 [C17414] -> 10k
- R_HV_LED1: value 4.7k_1%_1206 [C17936] -> 22k 1206
- R_HV_PD1: value 47k_1%_0805 [C17713] -> 47k
- TH1, TH2, TH3, TH4, TH5, TH6, TH7: value MF52A103J3950_10k [C123378] -> 10k B3950 1%
- moved J4 202.0 mm to (275.0, 13.5)
- moved TH5 121.3 mm to (228.9, 80.2)
- moved TH7 110.6 mm to (228.9, 179.4)
- moved J2 85.0 mm to (150.0, 150.0)
- moved J1 70.4 mm to (160.0, 87.5), turned to -90 degrees
- moved TH1 70.0 mm to (65.5, 30.6)
- moved TH2 69.3 mm to (65.5, 80.2)
- moved TH3 68.8 mm to (65.5, 129.8)
- moved TH4 68.5 mm to (65.5, 179.4)
- moved TH6 66.3 mm to (228.9, 129.8)
- moved J3 59.2 mm to (275.0, 41.0)
- moved R_HV_LED1 51.9 mm to (157.0, 38.0), turned to 180 degrees
- moved F_PTC15 46.7 mm to (127.0, 133.0)
- moved LED_HV1 45.7 mm to (152.0, 38.0)
- moved D_TVS13 45.2 mm to (141.0, 127.0), turned to -90 degrees
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Connections:
- net /03_BMS_Interface_and_Thermal/NTC_1_A renamed /03_BMS_Interface_and_Thermal/NTC1_A
- net /03_BMS_Interface_and_Thermal/NTC_1_B renamed /03_BMS_Interface_and_Thermal/NTC1_B
- net /03_BMS_Interface_and_Thermal/NTC_2_A renamed /03_BMS_Interface_and_Thermal/NTC2_A
- net /03_BMS_Interface_and_Thermal/NTC_2_B renamed /03_BMS_Interface_and_Thermal/NTC2_B
- net /03_BMS_Interface_and_Thermal/NTC_3_A renamed /03_BMS_Interface_and_Thermal/NTC3_A
- net /03_BMS_Interface_and_Thermal/NTC_3_B renamed /03_BMS_Interface_and_Thermal/NTC3_B
- net /03_BMS_Interface_and_Thermal/NTC_4_A renamed /03_BMS_Interface_and_Thermal/NTC4_A
- net /03_BMS_Interface_and_Thermal/NTC_4_B renamed /03_BMS_Interface_and_Thermal/NTC4_B
- net /03_BMS_Interface_and_Thermal/NTC_5_A renamed /03_BMS_Interface_and_Thermal/NTC5_A
- net /03_BMS_Interface_and_Thermal/NTC_5_B renamed /03_BMS_Interface_and_Thermal/NTC5_B
- net /03_BMS_Interface_and_Thermal/NTC_6_A renamed /03_BMS_Interface_and_Thermal/NTC6_A
- net /03_BMS_Interface_and_Thermal/NTC_6_B renamed /03_BMS_Interface_and_Thermal/NTC6_B
- net /03_BMS_Interface_and_Thermal/NTC_7_A renamed /03_BMS_Interface_and_Thermal/NTC7_A
- net /03_BMS_Interface_and_Thermal/NTC_7_B renamed /03_BMS_Interface_and_Thermal/NTC7_B
- net GND renamed PACK_NEG
- net Net-(Q_HV1-PadB) renamed /04_Power_Path_and_Protection/HV_BASE
- BT14 pad 1: CELL_14 -> CELL_14_UNFUSED
- D_TVS1 pad 1: /03_BMS_Interface_and_Thermal/BMS_V1 -> /03_BMS_Interface_and_Thermal/BMS_V0
- D_TVS1 pad 2: /03_BMS_Interface_and_Thermal/BMS_V0 -> /03_BMS_Interface_and_Thermal/BMS_V1
- D_TVS10 pad 1: /03_BMS_Interface_and_Thermal/BMS_V10 -> /03_BMS_Interface_and_Thermal/BMS_V9
- D_TVS10 pad 2: /03_BMS_Interface_and_Thermal/BMS_V9 -> /03_BMS_Interface_and_Thermal/BMS_V10
- D_TVS11 pad 1: /03_BMS_Interface_and_Thermal/BMS_V11 -> /03_BMS_Interface_and_Thermal/BMS_V10
- D_TVS11 pad 2: /03_BMS_Interface_and_Thermal/BMS_V10 -> /03_BMS_Interface_and_Thermal/BMS_V11
- D_TVS12 pad 1: /03_BMS_Interface_and_Thermal/BMS_V12 -> /03_BMS_Interface_and_Thermal/BMS_V11
- D_TVS12 pad 2: /03_BMS_Interface_and_Thermal/BMS_V11 -> /03_BMS_Interface_and_Thermal/BMS_V12
- D_TVS13 pad 1: /03_BMS_Interface_and_Thermal/BMS_V13 -> /03_BMS_Interface_and_Thermal/BMS_V12
- D_TVS13 pad 2: /03_BMS_Interface_and_Thermal/BMS_V12 -> /03_BMS_Interface_and_Thermal/BMS_V13
- D_TVS14 pad 1: /03_BMS_Interface_and_Thermal/BMS_V14 -> /03_BMS_Interface_and_Thermal/BMS_V13
- D_TVS14 pad 2: /03_BMS_Interface_and_Thermal/BMS_V13 -> /03_BMS_Interface_and_Thermal/BMS_V14
- D_TVS2 pad 1: /03_BMS_Interface_and_Thermal/BMS_V2 -> /03_BMS_Interface_and_Thermal/BMS_V1
- D_TVS2 pad 2: /03_BMS_Interface_and_Thermal/BMS_V1 -> /03_BMS_Interface_and_Thermal/BMS_V2
- D_TVS3 pad 1: /03_BMS_Interface_and_Thermal/BMS_V3 -> /03_BMS_Interface_and_Thermal/BMS_V2
- D_TVS3 pad 2: /03_BMS_Interface_and_Thermal/BMS_V2 -> /03_BMS_Interface_and_Thermal/BMS_V3
- D_TVS4 pad 1: /03_BMS_Interface_and_Thermal/BMS_V4 -> /03_BMS_Interface_and_Thermal/BMS_V3
- D_TVS4 pad 2: /03_BMS_Interface_and_Thermal/BMS_V3 -> /03_BMS_Interface_and_Thermal/BMS_V4
- D_TVS5 pad 1: /03_BMS_Interface_and_Thermal/BMS_V5 -> /03_BMS_Interface_and_Thermal/BMS_V4
- D_TVS5 pad 2: /03_BMS_Interface_and_Thermal/BMS_V4 -> /03_BMS_Interface_and_Thermal/BMS_V5
- D_TVS6 pad 1: /03_BMS_Interface_and_Thermal/BMS_V6 -> /03_BMS_Interface_and_Thermal/BMS_V5
- D_TVS6 pad 2: /03_BMS_Interface_and_Thermal/BMS_V5 -> /03_BMS_Interface_and_Thermal/BMS_V6
- D_TVS7 pad 1: /03_BMS_Interface_and_Thermal/BMS_V7 -> /03_BMS_Interface_and_Thermal/BMS_V6
- D_TVS7 pad 2: /03_BMS_Interface_and_Thermal/BMS_V6 -> /03_BMS_Interface_and_Thermal/BMS_V7
- D_TVS8 pad 1: /03_BMS_Interface_and_Thermal/BMS_V8 -> /03_BMS_Interface_and_Thermal/BMS_V7
- D_TVS8 pad 2: /03_BMS_Interface_and_Thermal/BMS_V7 -> /03_BMS_Interface_and_Thermal/BMS_V8
- D_TVS9 pad 1: /03_BMS_Interface_and_Thermal/BMS_V9 -> /03_BMS_Interface_and_Thermal/BMS_V8
- D_TVS9 pad 2: /03_BMS_Interface_and_Thermal/BMS_V8 -> /03_BMS_Interface_and_Thermal/BMS_V9
- F1 pad 1: CELL_16_UNFUSED -> CELL_14_UNFUSED
- F_PTC15 pad 1: CELL_14 -> CELL_14_UNFUSED
- R_HV_BASE1 pad 1: Net-(D_ZENER_HV1-K) -> /04_Power_Path_and_Protection/HV_Z_A
- R_HV_LED1 pad 2: Net-(LED_HV1-K) -> Net-(LED_HV1-A)
Routing:
- net PACK_NEG: track 725.1 -> 219.9 mm, vias 1 -> 5
- net CELL_15: track 418.3 -> 0.00 mm, vias 7 -> 0
- net CELL_14: track 320.8 -> 0.00 mm, vias 7 -> 0
- net CELL_16_UNFUSED: track 298.4 -> 0.00 mm, vias 1 -> 0
- net PACK_POS: track 394.5 -> 100.9 mm, vias 1 -> 0
- net CELL_14_UNFUSED: track 0.00 -> 267.6 mm, vias 0 -> 3
- net CELL_3: track 317.9 -> 129.4 mm, vias 7 -> 2
- net CELL_1: track 354.0 -> 171.0 mm, vias 7 -> 2
- net /03_BMS_Interface_and_Thermal/NTC1_B: track 29.5 -> 203.8 mm, vias 1 -> 0
- net /03_BMS_Interface_and_Thermal/NTC1_A: track 34.5 -> 206.4 mm, vias 1 -> 0
- net /03_BMS_Interface_and_Thermal/BMS_V16: track 148.2 -> 0.00 mm, vias 1 -> 0
- net /03_BMS_Interface_and_Thermal/BMS_V15: track 145.2 -> 0.00 mm, vias 1 -> 0
- net CELL_7: track 327.0 -> 189.6 mm, vias 7 -> 2
- net CELL_5: track 281.8 -> 148.0 mm, vias 7 -> 2
- net CELL_13: track 363.0 -> 243.0 mm, vias 7 -> 2
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- added copper zone on B.Cu, net CELL_14_UNFUSED
- added copper zone on F.Cu, net CELL_14_UNFUSED
- removed copper zone on B.Cu, net CELL_14
- removed copper zone on F.Cu, net CELL_14
- removed copper zone on B.Cu, net CELL_15
- removed copper zone on F.Cu, net CELL_15
- removed copper zone on B.Cu, net CELL_16_UNFUSED
- removed copper zone on F.Cu, net CELL_16_UNFUSED
Other:
- board text added: "+"
- board text added: "-"
- board text added: "14S 18650 BATTERY PACK BREAKOUT"
- board text added: "58.8V MAX | A4 297 x 210 mm | 4-LAYER"
- board text added: "B-"
- board text added: "BMS CELL SENSE J1 (JST XH 15P)"
- board text added: "C1"
- board text added: "C10"
- board text added: "C11"
- board text added: "C12"
- board text added: "C13"
- board text added: "C14"
- board text added: "C2"
- board text added: "C3"
- board text added: "C4"
- board text added: "C5"
- board text added: "C6"
- board text added: "C7"
- board text added: "C8"
- board text added: "C9"
- board text added: "CELL 8 (+) --> CELL 9 (-) BUS"
- board text added: "F1 5x20mm 10A"
- board text added: "FUSE BLOWN"
- board text added: "HV >44V"
- board text added: "NTC J2 (JST XH 14P)"
- board text added: "NTC1"
- board text added: "NTC2"
- board text added: "NTC3"
- board text added: "NTC4"
- board text added: "NTC5"
- board text added: "NTC6"
- board text added: "NTC7"
- board text added: "PACK+"
- board text added: "PACK-"
- board text added: "T1"
- board text added: "T2"
- board text added: "T3"
- board text added: "T4"
- board text added: "T5"
- board text added: "T6"
- board text added: "T7"
- board text added: "WARNING: LIVE 58.8V DC. INSERT CELLS WITH CORRECT POLARITY - RED LED = REVERSED CELL."
- board text removed: "BOTTOM PACK LINK: CELL 8(+) TO CELL 9(-)"
- board text removed: "DECIBELS LAB — MODULAR 16S / 14S BATTERY PACK ON PCB"
- board text removed: "F1: 20A CERAMIC FUSE (1500A DC BREAKING)"
- board text removed: "HV STROBE >42V DC"
- board text removed: "J1: BMS V-SENSE (1x17)"
- board text removed: "J2: BMS TEMP NTC (1x16)"
- board text removed: "PACK + (B+)"
- board text removed: "PACK - (GND)"
- board text removed: "REV 3.0 | TRUE A4 LANDSCAPE (297 x 210 mm) | 4-LAYER HEAVY COPPER (2oz/1oz/1oz/2oz) | ENIG FINISH"
- board text removed: "ROW 1: CELLS 1 TO 8 [SERPENTINE BUSBAR]"
- board text removed: "ROW 2: CELLS 16 TO 9 [SERPENTINE BUSBAR]"
- board text removed: "WARNING: LIVE BATTERY VOLTAGE UP TO 67.2V DC. CLASS 1 SELV COMPLIANT IN <=14S MODE. USE ACRYLIC COVER FOR 16S."

Commit message: Mirror the two cell columns (7+7) and move every external connector to the top edge
- Cells 1-7 down the left column, 8-14 up the right, identical row spacing;
  B- now lands at the top-left corner and cell 14+ at the top-right.
- Top edge, left to right: J2 NTC, B- lug, J1 balance (centred), PACK+ lug,
  5x20 fuse. Balance pin 1 = B- on the left, matching the cell order.
- PPTC/TVS sense block sits directly under J1; sense taps fan in on In1,
  NTC pairs run up to J2 on In2. NTCs renumbered along the series path.
- Pack TVS and HV indicator next to PACK+, PACK- return on a B.Cu strip.
- Mid-board M3 holes moved into the channel; wiring guide on silkscreen.
- ERC 0, DRC 0 (all severities), 0 unconnected, 0 parity issues.

Co-Authored-By: Claude Opus 5.5 <noreply@anthropic.com>
Claude-Session: https://claude.ai/code/session_01SDBUxKR8a94h5ECbt5NLbF
Parts:
- moved TP_N8 288.0 mm to (292.4, 199.1)
- moved TP_P8 288.0 mm to (292.4, 188.1)
- moved D_REV8 275.2 mm to (286.0, 188.6), turned to -90 degrees
- moved R_REV8 275.2 mm to (286.0, 198.6), turned to -90 degrees
- moved LED_REV8 275.0 mm to (286.0, 193.6), turned to -90 degrees
- moved J2 182.8 mm to (38.0, 5.50), turned to 0 degrees
- moved J4 171.0 mm to (104.0, 13.0)
- moved BT8 163.4 mm to (230.2, 192.6)
- moved TH7 125.5 mm to (231.5, 54.0), turned to 180 degrees
- moved D_TVS14 110.7 mm to (174.5, 24.0), turned to 0 degrees
- moved H5 110.1 mm to (127.0, 115.0)
- moved D_TVS13 101.4 mm to (170.5, 30.0), turned to 0 degrees
- moved D_TVS12 101.1 mm to (166.5, 24.0), turned to 0 degrees
- moved F_PTC15 101.0 mm to (176.5, 45.0), turned to 90 degrees
- moved F_PTC14 98.8 mm to (172.5, 38.0), turned to 90 degrees
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Routing:
- net CELL_7: track 189.6 -> 415.8 mm, vias 2 -> 6
- net CELL_14_UNFUSED: track 267.6 -> 97.4 mm, vias 3 -> 2
- net PACK_NEG: track 219.9 -> 50.1 mm, vias 5 -> 6
- net /03_BMS_Interface_and_Thermal/NTC5_A: track 171.3 -> 323.7 mm
- net /03_BMS_Interface_and_Thermal/NTC6_A: track 126.7 -> 269.1 mm
- net /03_BMS_Interface_and_Thermal/NTC5_B: track 173.7 -> 316.1 mm
- net /03_BMS_Interface_and_Thermal/NTC7_A: track 82.1 -> 214.5 mm
- net /03_BMS_Interface_and_Thermal/NTC6_B: track 129.1 -> 261.5 mm
- net CELL_5: track 148.0 -> 271.0 mm, vias 2 -> 3
- net /03_BMS_Interface_and_Thermal/NTC7_B: track 84.5 -> 206.9 mm
- net /03_BMS_Interface_and_Thermal/NTC1_A: track 206.4 -> 86.9 mm
- net /03_BMS_Interface_and_Thermal/NTC1_B: track 203.8 -> 85.7 mm
- net /03_BMS_Interface_and_Thermal/NTC4_B: track 96.5 -> 203.4 mm
- net /03_BMS_Interface_and_Thermal/NTC4_A: track 98.9 -> 204.6 mm
- net PACK_POS: track 100.9 -> 0.00 mm
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Other:
- board text added: "1. J1 <- BMS balance lead (B- wire on pin 1)"
- board text added: "2. J2 <- BMS NTC lead (or leave open)"
- board text added: "3. B- lug -> BMS B- PACK+ lug -> load/charger +"
- board text added: "4. Load/charger - -> BMS P-"
- board text added: "5. Insert cells LAST. A red LED = that cell is reversed."
- board text added: "B- / PACK-"
- board text added: "CELL 7 (+) --> CELL 8 (-) BUS"
- board text added: "F1 5x20 10A"
- board text added: "HOW TO CONNECT"
- board text added: "HV>44V"
- board text added: "J1 BALANCE -> BMS (1 = B- ... 15 = C14+)"
- board text added: "J2 NTC -> BMS (1-2 = NTC1 ... 13-14 = NTC7)"
- board text added: "Test loops: red = cell +, black = cell -"
- board text added: "to BMS B-"
- board text added: "to load / charger +"
- board text removed: "B-"
- board text removed: "BMS CELL SENSE J1 (JST XH 15P)"
- board text removed: "CELL 8 (+) --> CELL 9 (-) BUS"
- board text removed: "F1 5x20mm 10A"
- board text removed: "HV >44V"
- board text removed: "NTC J2 (JST XH 14P)"
- board text removed: "PACK-"
- board text removed: "T1"
- board text removed: "T2"
- board text removed: "T3"
- board text removed: "T4"
- board text removed: "T5"
- board text removed: "T6"
- board text removed: "T7"

Commit message: Senior-level layout rework: equal-resistance cell links, uniform pitch, sense spine
- Uniform 27.6 mm cell pitch (4.8 mm air gap around every cell).
- All 13 cell-to-cell links are identical copper straps (F.Cu + B.Cu); the
  cell 7->8 strap across the channel is widened to 16.15 mm so its
  resistance matches. 2-D field solve: 0.260 mOhm per link, 0.08 % spread
  (tools/acir.py, docs/acir_check.txt).
- Centre channel is now a sense spine: a 60 V PPTC at every node and one
  In1 bus into J1; per-cell TVS moved to SOD-323 (LKS05D3-B) directly under
  J1 so the whole BMS protection block sits on the top edge.
- Outer margins: per-cell test loops, reverse-cell LED, writable V/IR box.
- Top edge: B- lug, HV indicator + pack TVS, J1, J2, PACK+ lug, fuse.
- Shared geometry module (tools/geom.py) used by layout and ACIR check.
- ERC 0, DRC 0, 0 unconnected, 0 parity issues.

Co-Authored-By: Claude Opus 5.5 <noreply@anthropic.com>
Claude-Session: https://claude.ai/code/session_01SDBUxKR8a94h5ECbt5NLbF
Parts:
- D_TVS1, D_TVS10, D_TVS11, D_TVS12, D_TVS13, D_TVS14, D_TVS2, D_TVS3, D_TVS4, D_TVS5, D_TVS6, D_TVS7, D_TVS8, D_TVS9: value SMAJ5.0CA -> LKS05D3-B; footprint Diode_SMD:D_SMA -> Diode_SMD:D_SOD-323
- moved F_PTC8 145.6 mm to (140.4, 183.3)
- moved J2 135.0 mm to (173.0, 5.50)
- moved F_PTC7 129.5 mm to (140.4, 174.4)
- moved F_PTC9 129.5 mm to (156.6, 174.4)
- moved H5 116.2 mm to (12.0, 98.4)
- moved H6 116.2 mm to (285.0, 98.4)
- moved F_PTC10 115.4 mm to (156.6, 153.4), turned to -90 degrees
- moved F_PTC6 115.4 mm to (140.4, 153.4), turned to -90 degrees
- moved TH5 112.7 mm to (206.8, 43.2), turned to 0 degrees
- moved TH7 102.7 mm to (206.8, 153.6), turned to 0 degrees
- moved F_PTC1 97.3 mm to (26.0, 22.0)
- moved F_PTC15 97.3 mm to (271.0, 22.0)
- moved R_HV_LED1 91.2 mm to (115.3, 5.00)
- moved R_HV_PD1 90.5 mm to (102.5, 7.20)
- moved LED_HV1 90.5 mm to (111.0, 5.00)
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Routing:
- net /03_BMS_Interface_and_Thermal/NTC5_A: track 323.7 -> 59.9 mm
- net /03_BMS_Interface_and_Thermal/NTC5_B: track 316.1 -> 58.8 mm
- net CELL_7: track 415.8 -> 245.3 mm, vias 6 -> 10
- net /03_BMS_Interface_and_Thermal/NTC6_A: track 269.1 -> 112.9 mm
- net /03_BMS_Interface_and_Thermal/BMS_V7: track 30.4 -> 183.4 mm, vias 0 -> 2
- net /03_BMS_Interface_and_Thermal/NTC6_B: track 261.5 -> 111.8 mm
- net /03_BMS_Interface_and_Thermal/BMS_V8: track 38.0 -> 173.9 mm, vias 0 -> 2
- net /03_BMS_Interface_and_Thermal/BMS_V6: track 38.0 -> 173.9 mm, vias 0 -> 2
- net CELL_8: track 260.1 -> 127.1 mm, vias 2 -> 8
- net CELL_6: track 260.1 -> 127.1 mm, vias 2 -> 8
- net /03_BMS_Interface_and_Thermal/BMS_V5: track 31.6 -> 161.0 mm, vias 0 -> 2
- net /03_BMS_Interface_and_Thermal/BMS_V9: track 31.6 -> 161.0 mm, vias 0 -> 2
- net CELL_5: track 271.0 -> 147.5 mm, vias 3 -> 8
- net CELL_9: track 271.0 -> 147.5 mm, vias 3 -> 8
- net CELL_14_UNFUSED: track 97.4 -> 11.9 mm, vias 2 -> 0
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Other:
- board text added: "1. J1 <- BMS balance lead (B- wire = pin 1)"
- board text added: "2. J2 <- BMS NTC lead (optional)"
- board text added: "3. B- lug -> BMS B- | PACK+ lug -> load +"
- board text added: "4. Load / charger - -> BMS P-"
- board text added: "5. Insert cells LAST. Red LED = reversed cell"
- board text added: "58.8V MAX | A4 | 4-LAYER | EQUAL 0.26 mOhm CELL LINKS"
- board text added: "CELL 7 (+) -> CELL 8 (-)"
- board text added: "IR _____"
- board text added: "J1 BMS BALANCE 1 = B- ... 15 = C14+"
- board text added: "J2 BMS NTC 1-2 = NTC1 ... 13-14 = NTC7"
- board text added: "NTC1 C1/C2"
- board text added: "NTC2 C3/C4"
- board text added: "NTC3 C5/C6"
- board text added: "NTC4 C6/C7"
- board text added: "NTC5 C13/C14"
- board text added: "NTC6 C11/C12"
- board text added: "NTC7 C9/C10"
- board text added: "V ______"
- board text added: "WARNING: LIVE 58.8V DC - INSERT CELLS WITH CORRECT POLARITY - RED LED = REVERSED CELL"
- board text removed: "1. J1 <- BMS balance lead (B- wire on pin 1)"
- board text removed: "2. J2 <- BMS NTC lead (or leave open)"
- board text removed: "3. B- lug -> BMS B- PACK+ lug -> load/charger +"
- board text removed: "4. Load/charger - -> BMS P-"
- board text removed: "5. Insert cells LAST. A red LED = that cell is reversed."
- board text removed: "58.8V MAX | A4 297 x 210 mm | 4-LAYER"
- board text removed: "CELL 7 (+) --> CELL 8 (-) BUS"
- board text removed: "J1 BALANCE -> BMS (1 = B- ... 15 = C14+)"
- board text removed: "J2 NTC -> BMS (1-2 = NTC1 ... 13-14 = NTC7)"
- board text removed: "NTC1"
- board text removed: "NTC2"
- board text removed: "NTC3"
- board text removed: "NTC4"
- board text removed: "NTC5"
- board text removed: "NTC6"
- board text removed: "NTC7"
- board text removed: "Test loops: red = cell +, black = cell -"
- board text removed: "WARNING: LIVE 58.8V DC. INSERT CELLS WITH CORRECT POLARITY - RED LED = REVERSED CELL."

Commit message: Make the board mirror-symmetric about its centre line
- NTCs: 3 per side in mirrored gaps, NTC4 on the centre line at the
  cell 7->8 bus (J2 pins 7/8); J2 pin 2n-1/2n = NTCn kept.
- Sense spine exactly symmetric: tap-7 PPTC and its bus line on the centre
  line, side buses mirrored, J1 fan symmetric.
- Per-cell LED strings: series order chosen per cell so mirrored twins use
  the same parts in the same places (function unchanged).
- TVS chain under J1 mirrored; the centre pair stands vertically either side
  of lane 7.
- HV indicator + pack TVS centred at J2's mirror position; top-band copper
  mirrored; 4 corner fiducials.
- tools/symcheck.py audits mirror partners: only J2, the HV block and the
  single PACK+ fuse (+ its LED) are one-of-a-kind.
- ERC 0, DRC 0, 0 unconnected, 0 parity; ACIR spread 0.08 %.

Co-Authored-By: Claude Opus 5.5 <noreply@anthropic.com>
Claude-Session: https://claude.ai/code/session_01SDBUxKR8a94h5ECbt5NLbF
Parts:
- added FID4: Fiducial, Fiducial:Fiducial_1mm_Mask2mm, F.Cu at (283.0, 206.6)
- moved TH4 64.4 mm to (147.2, 205.6)
- moved D_REV1 10.0 mm to (31.0, 25.9)
- moved D_REV11 10.0 mm to (266.0, 115.7)
- moved D_REV13 10.0 mm to (266.0, 60.5)
- moved D_REV3 10.0 mm to (31.0, 81.1)
- moved D_REV5 10.0 mm to (31.0, 136.3)
- moved D_REV7 10.0 mm to (31.0, 191.5)
- moved D_REV9 10.0 mm to (266.0, 170.9)
- moved R_REV1 10.0 mm to (31.0, 35.9)
- moved R_REV11 10.0 mm to (266.0, 105.7)
- moved R_REV13 10.0 mm to (266.0, 50.5)
- moved R_REV3 10.0 mm to (31.0, 91.1)
- moved R_REV5 10.0 mm to (31.0, 146.3)
- moved R_REV7 10.0 mm to (31.0, 201.5)
- moved R_REV9 10.0 mm to (266.0, 160.9)
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Connections:
- D_REV1 pad 1: CELL_1 -> Net-(D_REV1-K)
- D_REV1 pad 2: Net-(D_REV1-A) -> PACK_NEG
- D_REV11 pad 1: CELL_11 -> Net-(D_REV11-K)
- D_REV11 pad 2: Net-(D_REV11-A) -> CELL_10
- D_REV13 pad 1: CELL_13 -> Net-(D_REV13-K)
- D_REV13 pad 2: Net-(D_REV13-A) -> CELL_12
- D_REV3 pad 1: CELL_3 -> Net-(D_REV3-K)
- D_REV3 pad 2: Net-(D_REV3-A) -> CELL_2
- D_REV5 pad 1: CELL_5 -> Net-(D_REV5-K)
- D_REV5 pad 2: Net-(D_REV5-A) -> CELL_4
- D_REV7 pad 1: CELL_7 -> Net-(D_REV7-K)
- D_REV7 pad 2: Net-(D_REV7-A) -> CELL_6
- D_REV9 pad 1: CELL_9 -> Net-(D_REV9-K)
- D_REV9 pad 2: Net-(D_REV9-A) -> CELL_8
- LED_REV1 pad 1: Net-(D_REV1-A) -> Net-(LED_REV1-K)
- LED_REV1 pad 2: Net-(LED_REV1-A) -> Net-(D_REV1-K)
- LED_REV11 pad 1: Net-(D_REV11-A) -> Net-(LED_REV11-K)
- LED_REV11 pad 2: Net-(LED_REV11-A) -> Net-(D_REV11-K)
- LED_REV13 pad 1: Net-(D_REV13-A) -> Net-(LED_REV13-K)
- LED_REV13 pad 2: Net-(LED_REV13-A) -> Net-(D_REV13-K)
- LED_REV3 pad 1: Net-(D_REV3-A) -> Net-(LED_REV3-K)
- LED_REV3 pad 2: Net-(LED_REV3-A) -> Net-(D_REV3-K)
- LED_REV5 pad 1: Net-(D_REV5-A) -> Net-(LED_REV5-K)
- LED_REV5 pad 2: Net-(LED_REV5-A) -> Net-(D_REV5-K)
- LED_REV7 pad 1: Net-(D_REV7-A) -> Net-(LED_REV7-K)
- LED_REV7 pad 2: Net-(LED_REV7-A) -> Net-(D_REV7-K)
- LED_REV9 pad 1: Net-(D_REV9-A) -> Net-(LED_REV9-K)
- LED_REV9 pad 2: Net-(LED_REV9-A) -> Net-(D_REV9-K)
- R_REV1 pad 1: Net-(LED_REV1-A) -> CELL_1
- R_REV1 pad 2: PACK_NEG -> Net-(LED_REV1-K)
- R_REV11 pad 1: Net-(LED_REV11-A) -> CELL_11
- R_REV11 pad 2: CELL_10 -> Net-(LED_REV11-K)
- R_REV13 pad 1: Net-(LED_REV13-A) -> CELL_13
- R_REV13 pad 2: CELL_12 -> Net-(LED_REV13-K)
- R_REV3 pad 1: Net-(LED_REV3-A) -> CELL_3
- R_REV3 pad 2: CELL_2 -> Net-(LED_REV3-K)
- R_REV5 pad 1: Net-(LED_REV5-A) -> CELL_5
- R_REV5 pad 2: CELL_4 -> Net-(LED_REV5-K)
- R_REV7 pad 1: Net-(LED_REV7-A) -> CELL_7
- R_REV7 pad 2: CELL_6 -> Net-(LED_REV7-K)
- R_REV9 pad 1: Net-(LED_REV9-A) -> CELL_9
- R_REV9 pad 2: CELL_8 -> Net-(LED_REV9-K)
Routing:
- net /03_BMS_Interface_and_Thermal/NTC4_B: track 278.7 -> 241.7 mm
- net /03_BMS_Interface_and_Thermal/NTC4_A: track 276.1 -> 240.5 mm
- net /03_BMS_Interface_and_Thermal/BMS_V7: track 183.4 -> 177.9 mm
- net Net-(LED_REV9-A): track 3.15 -> 0.00 mm
- net Net-(LED_REV7-A): track 3.15 -> 0.00 mm
- net Net-(LED_REV5-K): track 0.00 -> 3.15 mm
- net Net-(LED_REV5-A): track 3.15 -> 0.00 mm
- net Net-(LED_REV3-A): track 3.15 -> 0.00 mm
- net Net-(LED_REV13-K): track 0.00 -> 3.15 mm
- net Net-(LED_REV11-K): track 0.00 -> 3.15 mm
- net Net-(LED_REV11-A): track 3.15 -> 0.00 mm
- net Net-(LED_REV1-A): track 3.15 -> 0.00 mm
- net Net-(LED_REV13-A): track 3.15 -> 0.00 mm
- net Net-(LED_REV1-K): track 0.00 -> 3.15 mm
- net Net-(LED_REV3-K): track 0.00 -> 3.15 mm
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Other:
- board text added: "J2 BMS NTC (7 sensors)"
- board text added: "NTC4 BUS"
- board text added: "pins 2n-1 / 2n = NTCn | NTC4 = centre bus"
- board text removed: "J2 BMS NTC 1-2 = NTC1 ... 13-14 = NTC7"
- board text removed: "NTC4 C6/C7"
