File: BatteryPack_16S_A4_Breakout.kicad_pcb (KiCad board)
At the start: 4 copper layers, 297 x 210 mm, 144 parts, among them J1 B15B-XH-A, J2 B14B-XH-A, J3 PACK+ M4, J4 PACK- M4

Commit message: just tested
Parts:
- moved TP_P13 109.7 mm to (155.7, 87.1)
- moved TP_N14 104.8 mm to (156.6, 50.5)
Routing:
- net CELL_13: track 147.7 -> 124.4 mm
